Commit message: feat: update scout drone urdf with spinning propeller joints
Replaced the rigid scout_drone.urdf and meshes with the newly generated versions containing the continuous propeller joints. Re-mapped the mesh paths inside the URDF to point to the correct package directories.

File: src/opsg_description/urdf/scout_drone.urdf (robot description, URDF)
Before this commit: robot cad, 21 links, 20 joints
Links:
- added link propeller, mass 1e-09
- added link propeller_2, mass 1e-09
- added link propeller_2_propeller_2, mass 0.009; collision mesh filename=package://opsg_description/meshes/scout_drone/propeller.stl; visual mesh filename=package://opsg_description/meshes/scout_drone/propeller.stl
- added link propeller_3, mass 1e-09
- added link propeller_3_propeller_3, mass 0.009; collision mesh filename=package://opsg_description/meshes/scout_drone/propeller.stl; visual mesh filename=package://opsg_description/meshes/scout_drone/propeller.stl
- added link propeller_4, mass 1e-09
- added link propeller_4_propeller_4, mass 0.009; collision mesh filename=package://opsg_description/meshes/scout_drone/propeller.stl; visual mesh filename=package://opsg_description/meshes/scout_drone/propeller.stl
- added link propeller_propeller, mass 0.009; collision mesh filename=package://opsg_description/meshes/scout_drone/propeller.stl; visual mesh filename=package://opsg_description/meshes/scout_drone/propeller.stl
Joints:
- added joint prop1: type revolute, parent bottom_plate, child propeller, origin xyz=-0.12 -0.2 0.022 rpy=3.14159 -0 0, axis 0 0 1, limit lower=-3.141592653589793 upper=3.141592653589793 effort=10 velocity=10
- added joint prop2: type revolute, parent bottom_plate, child propeller_2, origin xyz=-0.16 0.09 0.022 rpy=3.14159 -0 0, axis 0 0 1, limit lower=-3.141592653589793 upper=3.141592653589793 effort=10 velocity=10
- added joint prop3: type revolute, parent bottom_plate, child propeller_3, origin xyz=0.16 0.09 0.022 rpy=3.14159 -0 0, axis 0 0 1, limit lower=-3.141592653589793 upper=3.141592653589793 effort=10 velocity=10
- added joint prop4: type revolute, parent bottom_plate, child propeller_4, origin xyz=0.12 -0.2 0.022 rpy=3.14159 -0 0, axis 0 0 1, limit lower=-3.141592653589793 upper=3.141592653589793 effort=10 velocity=10
- added joint propeller_2_propeller_2_fixed: type fixed, parent propeller_2, child propeller_2_propeller_2, origin xyz=0.12 -0.2 0.022 rpy=3.14159 -0 0, axis 0 0 1, limit effort=10 velocity=10
- added joint propeller_3_propeller_3_fixed: type fixed, parent propeller_3, child propeller_3_propeller_3, origin xyz=0.12 -0.2 0.022 rpy=3.14159 -0 0, axis 0 0 1, limit effort=10 velocity=10
- added joint propeller_4_propeller_4_fixed: type fixed, parent propeller_4, child propeller_4_propeller_4, origin xyz=0.12 -0.2 0.022 rpy=3.14159 -0 0, axis 0 0 1, limit effort=10 velocity=10
- added joint propeller_propeller_fixed: type fixed, parent propeller, child propeller_propeller, origin xyz=0.12 -0.2 0.022 rpy=3.14159 -0 0, axis 0 0 1, limit effort=10 velocity=10

Commit message: fix: add dummy base_link to scout drone urdf
Added a weightless dummy base_link connected to the bottom_plate via a fixed joint. This resolves the kdl_parser warning where the root link is not allowed to have mass or inertia.

File: src/opsg_description/urdf/scout_drone.urdf (robot description, URDF)
Before this commit: robot scout_drone, 29 links, 28 joints
Links:
- added link base_link
Joints:
- added joint base_joint: type fixed, parent base_link, child bottom_plate, origin xyz=0 0 0 rpy=0 0 0
